File: board/hoatzin.kicad_pcb (KiCad board)
At the start: 4 copper layers, 221 x 71.5 mm, 61 parts, among them J1 2-215079-0, J10 Conn_01x03_Male, J11 Conn_01x03_Male, J12 Conn_01x02_Male, J13 Conn_01x02_Male, J14 Conn_01x03_Male, J15 Conn_01x04_Male, J16 Conn_01x02_Male, J2 2-215079-0, J3 671-0501, J4 671-0501, J5 671-0501, J6 292304-1, J7 0702462004, J8 SN37A14B, J9 SN37A14B, U1 STM32L476RGT6, U2 6N139, U3 SN74LS14D, U4 LD3985M33R_SOT23

Commit message: created firmware project. Tested MIDI communication over MIDI port as well as USB MIDI
Parts:
- D2: value BAT60AE6327H -> BAT60AE6327HTSA1
- FB1: value GZ2012D601TF -> HZ0805E601R-10
