File: board/keyConn.kicad_sch (KiCad schematic)
At the start: 4 parts, among them J1 2-215079-0, J15 Conn_01x04_Male, J2 2-215079-0

Commit message: created firmware project. Tested MIDI communication over MIDI port as well as USB MIDI
Parts:
- J1, J2: Digi-Key Part Number (none) -> A111123CT-ND
- J15: Digi-Key Part Number (none) -> HTSW-104-14-TM-S-ND
- R20: Digi-Key Part Number (none) -> P1.00KCCT-ND; LCSC C17513 -> (none); MANUFACTURER UNI-ROYAL(Uniroyal Elec) -> Panasonic Electronic Components; Manufacturer_Name UNI-ROYAL(Uniroyal Elec) -> Panasonic Electronic Components; Manufacturer_Part_Number 0805W8F1001T5E -> ERJ-6ENF1001V
Changed lines of the file:
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@@
+      (effects (font (size 1.27 1.27)) hide)
+    )
+    (property "Digi-Key Part Number" "HTSW-104-14-TM-S-ND" (id 8) (at 86.36 93.98 0)
       (effects (font (size 1.27 1.27)) hide)
     )
@@
     )
     (property "Manufacturer_Part_Number" "2-215079-0" (id 7) (at 229.87 66.04 0)
+      (effects (font (size 1.27 1.27)) hide)
+    )
+    (property "Digi-Key Part Number" "A111123CT-ND" (id 8) (at 229.87 66.04 0)
       (effects (font (size 1.27 1.27)) hide)
     )
@@
       (effects (font (size 1.27 1.27)) hide)
     )
+    (property "Digi-Key Part Number" "A111123CT-ND" (id 8) (at 151.13 66.04 0)
+      (effects (font (size 1.27 1.27)) hide)
+    )
     (pin "1")
     (pin "10")
@@
       (effects (font (size 1.27 1.27)) hide)
     )
-    (property "Datasheet" "https://datasheet.lcsc.com/lcsc/2205311800_UNI-ROYAL-Uniroyal-Elec-0805W8F1001T5E_C17513.pdf" (id 3) (at 67.31 86.36 0)
+    (property "Datasheet" "" (id 3) (at 67.31 86.36 0)
       (effects (font (size 1.27 1.27)) hide)
     )
@@
       (effects (font (size 1.27 1.27)) hide)
     )
-    (property "MANUFACTURER" "UNI-ROYAL(Uniroyal Elec)" (id 5) (at 67.31 86.36 0)
+    (property "MANUFACTURER" "Panasonic Electronic Components" (id 5) (at 67.31 86.36 0)
       (effects (font (size 1.27 1.27)) hide)
     )
-    (property "Manufacturer_Name" "UNI-ROYAL(Uniroyal Elec)" (id 6) (at 67.31 86.36 0)
+    (property "Manufacturer_Name" "Panasonic Electronic Components" (id 6) (at 67.31 86.36 0)
       (effects (font (size 1.27 1.27)) hide)
     )
-    (property "Manufacturer_Part_Number" "0805W8F1001T5E" (id 7) (at 67.31 86.36 0)
+    (property "Manufacturer_Part_Number" "ERJ-6ENF1001V" (id 7) (at 67.31 86.36 0)
       (effects (font (size 1.27 1.27)) hide)
     )
-    (property "LCSC" "C17513" (id 8) (at 67.31 86.36 0)
+    (property "LCSC" "" (id 8) (at 67.31 86.36 0)
       (effects (font (size 1.27 1.27)) hide)
     )
+    (property "Digi-Key Part Number" "P1.00KCCT-ND" (id 9) (at 67.31 86.36 0)
+      (effects (font (size 1.27 1.27)) hide)
+    )
