File: board/pedalConn.kicad_sch (KiCad schematic)
At the start: 8 parts, among them J8 SN37A14B, J9 SN37A14B

Commit message: created firmware project. Tested MIDI communication over MIDI port as well as USB MIDI
Parts:
- J8, J9: Digi-Key Part Number (none) -> SC1570-ND
- R10, R11, R12, R13, R14, R15: Digi-Key Part Number (none) -> P1.00KCCT-ND; LCSC C17513 -> (none); MANUFACTURER UNI-ROYAL(Uniroyal Elec) -> Panasonic Electronic Components; Manufacturer_Name UNI-ROYAL(Uniroyal Elec) -> Panasonic Electronic Components; Manufacturer_Part_Number 0805W8F1001T5E -> ERJ-6ENF1001V
Changed lines of the file:
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@@
       (effects (font (size 1.27 1.27)) hide)
     )
-    (property "Datasheet" "https://datasheet.lcsc.com/lcsc/2205311800_UNI-ROYAL-Uniroyal-Elec-0805W8F1001T5E_C17513.pdf" (id 3) (at 85.09 119.38 0)
+    (property "Datasheet" "" (id 3) (at 85.09 119.38 0)
       (effects (font (size 1.27 1.27)) hide)
     )
@@
       (effects (font (size 1.27 1.27)) hide)
     )
-    (property "MANUFACTURER" "UNI-ROYAL(Uniroyal Elec)" (id 5) (at 85.09 119.38 0)
-      (effects (font (size 1.27 1.27)) hide)
-    )
-    (property "Manufacturer_Name" "UNI-ROYAL(Uniroyal Elec)" (id 6) (at 85.09 119.38 0)
-      (effects (font (size 1.27 1.27)) hide)
-    )
-    (property "Manufacturer_Part_Number" "0805W8F1001T5E" (id 7) (at 85.09 119.38 0)
-      (effects (font (size 1.27 1.27)) hide)
-    )
-    (property "LCSC" "C17513" (id 8) (at 85.09 119.38 0)
+    (property "MANUFACTURER" "Panasonic Electronic Components" (id 5) (at 85.09 119.38 0)
+      (effects (font (size 1.27 1.27)) hide)
+    )
+    (property "Manufacturer_Name" "Panasonic Electronic Components" (id 6) (at 85.09 119.38 0)
+      (effects (font (size 1.27 1.27)) hide)
+    )
+    (property "Manufacturer_Part_Number" "ERJ-6ENF1001V" (id 7) (at 85.09 119.38 0)
+      (effects (font (size 1.27 1.27)) hide)
+    )
+    (property "LCSC" "" (id 8) (at 85.09 119.38 0)
+      (effects (font (size 1.27 1.27)) hide)
+    )
+    (property "Digi-Key Part Number" "P1.00KCCT-ND" (id 9) (at 85.09 119.38 0)
       (effects (font (size 1.27 1.27)) hide)
     )
@@
       (effects (font (size 1.27 1.27)) hide)
     )
-    (property "Datasheet" "https://datasheet.lcsc.com/lcsc/2205311800_UNI-ROYAL-Uniroyal-Elec-0805W8F1001T5E_C17513.pdf" (id 3) (at 168.91 119.38 0)
+    (property "Datasheet" "" (id 3) (at 168.91 119.38 0)
       (effects (font (size 1.27 1.27)) hide)
     )
@@
       (effects (font (size 1.27 1.27)) hide)
     )
-    (property "MANUFACTURER" "UNI-ROYAL(Uniroyal Elec)" (id 5) (at 168.91 119.38 0)
-      (effects (font (size 1.27 1.27)) hide)
-    )
-    (property "Manufacturer_Name" "UNI-ROYAL(Uniroyal Elec)" (id 6) (at 168.91 119.38 0)
-      (effects (font (size 1.27 1.27)) hide)
-    )
-    (property "Manufacturer_Part_Number" "0805W8F1001T5E" (id 7) (at 168.91 119.38 0)
-      (effects (font (size 1.27 1.27)) hide)
-    )
-    (property "LCSC" "C17513" (id 8) (at 168.91 119.38 0)
+    (property "MANUFACTURER" "Panasonic Electronic Components" (id 5) (at 168.91 119.38 0)
+      (effects (font (size 1.27 1.27)) hide)
+    )
+    (property "Manufacturer_Name" "Panasonic Electronic Components" (id 6) (at 168.91 119.38 0)
+      (effects (font (size 1.27 1.27)) hide)
+    )
+    (property "Manufacturer_Part_Number" "ERJ-6ENF1001V" (id 7) (at 168.91 119.38 0)
+      (effects (font (size 1.27 1.27)) hide)
+    )
+    (property "LCSC" "" (id 8) (at 168.91 119.38 0)
+      (effects (font (size 1.27 1.27)) hide)
+    )
+    (property "Digi-Key Part Number" "P1.00KCCT-ND" (id 9) (at 168.91 119.38 0)
       (effects (font (size 1.27 1.27)) hide)
     )
@@
     )
     (property "MANUFACTURER" "Switchcraft" (id 12) (at 125.73 104.14 0)
+      (effects (font (size 1.27 1.27)) hide)
+    )
+    (property "Digi-Key Part Number" "SC1570-ND" (id 13) (at 125.73 104.14 0)
       (effects (font (size 1.27 1.27)) hide)
     )
@@
       (effects (font (size 1.27 1.27)) hide)
     )
-    (property "Datasheet" "https://datasheet.lcsc.com/lcsc/2205311800_UNI-ROYAL-Uniroyal-Elec-0805W8F1001T5E_C17513.pdf" (id 3) (at 90.17 119.38 0)
+    (property "Datasheet" "" (id 3) (at 90.17 119.38 0)
       (effects (font (size 1.27 1.27)) hide)
     )
@@
       (effects (font (size 1.27 1.27)) hide)
     )
-    (property "MANUFACTURER" "UNI-ROYAL(Uniroyal Elec)" (id 5) (at 90.17 119.38 0)
-      (effects (font (size 1.27 1.27)) hide)
-    )
-    (property "Manufacturer_Name" "UNI-ROYAL(Uniroyal Elec)" (id 6) (at 90.17 119.38 0)
-      (effects (font (size 1.27 1.27)) hide)
-    )
-    (property "Manufacturer_Part_Number" "0805W8F1001T5E" (id 7) (at 90.17 119.38 0)
-      (effects (font (size 1.27 1.27)) hide)
-    )
-    (property "LCSC" "C17513" (id 8) (at 90.17 119.38 0)
+    (property "MANUFACTURER" "Panasonic Electronic Components" (id 5) (at 90.17 119.38 0)
+      (effects (font (size 1.27 1.27)) hide)
+    )
+    (property "Manufacturer_Name" "Panasonic Electronic Components" (id 6) (at 90.17 119.38 0)
+      (effects (font (size 1.27 1.27)) hide)
+    )
+    (property "Manufacturer_Part_Number" "ERJ-6ENF1001V" (id 7) (at 90.17 119.38 0)
+      (effects (font (size 1.27 1.27)) hide)
+    )
+    (property "LCSC" "" (id 8) (at 90.17 119.38 0)
+      (effects (font (size 1.27 1.27)) hide)
+    )
+    (property "Digi-Key Part Number" "P1.00KCCT-ND" (id 9) (at 90.17 119.38 0)
       (effects (font (size 1.27 1.27)) hide)
     )
@@
       (effects (font (size 1.27 1.27)) hide)
     )
-    (property "Datasheet" "https://datasheet.lcsc.com/lcsc/2205311800_UNI-ROYAL-Uniroyal-Elec-0805W8F1001T5E_C17513.pdf" (id 3) (at 168.91 86.36 0)
+    (property "Datasheet" "" (id 3) (at 168.91 86.36 0)
       (effects (font (size 1.27 1.27)) hide)
     )
@@
       (effects (font (size 1.27 1.27)) hide)
     )
-    (property "MANUFACTURER" "UNI-ROYAL(Uniroyal Elec)" (id 5) (at 168.91 86.36 0)
-      (effects (font (size 1.27 1.27)) hide)
-    )
-    (property "Manufacturer_Name" "UNI-ROYAL(Uniroyal Elec)" (id 6) (at 168.91 86.36 0)
-      (effects (font (size 1.27 1.27)) hide)
-    )
-    (property "Manufacturer_Part_Number" "0805W8F1001T5E" (id 7) (at 168.91 86.36 0)
-      (effects (font (size 1.27 1.27)) hide)
-    )
-    (property "LCSC" "C17513" (id 8) (at 168.91 86.36 0)
+    (property "MANUFACTURER" "Panasonic Electronic Components" (id 5) (at 168.91 86.36 0)
+      (effects (font (size 1.27 1.27)) hide)
+    )
+    (property "Manufacturer_Name" "Panasonic Electronic Components" (id 6) (at 168.91 86.36 0)
+      (effects (font (size 1.27 1.27)) hide)
+    )
+    (property "Manufacturer_Part_Number" "ERJ-6ENF1001V" (id 7) (at 168.91 86.36 0)
+      (effects (font (size 1.27 1.27)) hide)
+    )
+    (property "LCSC" "" (id 8) (at 168.91 86.36 0)
+      (effects (font (size 1.27 1.27)) hide)
+    )
+    (property "Digi-Key Part Number" "P1.00KCCT-ND" (id 9) (at 168.91 86.36 0)
       (effects (font (size 1.27 1.27)) hide)
     )
@@
     )
     (property "MANUFACTURER" "Switchcraft" (id 12) (at 41.91 104.14 0)
+      (effects (font (size 1.27 1.27)) hide)
+    )
+    (property "Digi-Key Part Number" "SC1570-ND" (id 13) (at 41.91 104.14 0)
       (effects (font (size 1.27 1.27)) hide)
     )
@@
       (effects (font (size 1.27 1.27)) hide)
     )
-    (property "Datasheet" "https://datasheet.lcsc.com/lcsc/2205311800_UNI-ROYAL-Uniroyal-Elec-0805W8F1001T5E_C17513.pdf" (id 3) (at 90.17 86.36 0)
+    (property "Datasheet" "" (id 3) (at 90.17 86.36 0)
       (effects (font (size 1.27 1.27)) hide)
     )
@@
       (effects (font (size 1.27 1.27)) hide)
     )
-    (property "MANUFACTURER" "UNI-ROYAL(Uniroyal Elec)" (id 5) (at 90.17 86.36 0)
-      (effects (font (size 1.27 1.27)) hide)
-    )
-    (property "Manufacturer_Name" "UNI-ROYAL(Uniroyal Elec)" (id 6) (at 90.17 86.36 0)
-      (effects (font (size 1.27 1.27)) hide)
-    )
-    (property "Manufacturer_Part_Number" "0805W8F1001T5E" (id 7) (at 90.17 86.36 0)
-      (effects (font (size 1.27 1.27)) hide)
-    )
-    (property "LCSC" "C17513" (id 8) (at 90.17 86.36 0)
+    (property "MANUFACTURER" "Panasonic Electronic Components" (id 5) (at 90.17 86.36 0)
+      (effects (font (size 1.27 1.27)) hide)
+    )
+    (property "Manufacturer_Name" "Panasonic Electronic Components" (id 6) (at 90.17 86.36 0)
+      (effects (font (size 1.27 1.27)) hide)
+    )
+    (property "Manufacturer_Part_Number" "ERJ-6ENF1001V" (id 7) (at 90.17 86.36 0)
+      (effects (font (size 1.27 1.27)) hide)
+    )
+    (property "LCSC" "" (id 8) (at 90.17 86.36 0)
+      (effects (font (size 1.27 1.27)) hide)
+    )
+    (property "Digi-Key Part Number" "P1.00KCCT-ND" (id 9) (at 90.17 86.36 0)
       (effects (font (size 1.27 1.27)) hide)
     )
@@
       (effects (font (size 1.27 1.27)) hide)
     )
-    (property "Datasheet" "https://datasheet.lcsc.com/lcsc/2205311800_UNI-ROYAL-Uniroyal-Elec-0805W8F1001T5E_C17513.pdf" (id 3) (at 85.09 86.36 0)
+    (property "Datasheet" "" (id 3) (at 85.09 86.36 0)
       (effects (font (size 1.27 1.27)) hide)
     )
@@
       (effects (font (size 1.27 1.27)) hide)
     )
-    (property "MANUFACTURER" "UNI-ROYAL(Uniroyal Elec)" (id 5) (at 85.09 86.36 0)
-      (effects (font (size 1.27 1.27)) hide)
-    )
-    (property "Manufacturer_Name" "UNI-ROYAL(Uniroyal Elec)" (id 6) (at 85.09 86.36 0)
-      (effects (font (size 1.27 1.27)) hide)
-    )
-    (property "Manufacturer_Part_Number" "0805W8F1001T5E" (id 7) (at 85.09 86.36 0)
-      (effects (font (size 1.27 1.27)) hide)
-    )
-    (property "LCSC" "C17513" (id 8) (at 85.09 86.36 0)
-      (effects (font (size 1.27 1.27)) hide)
-    )
+    (property "MANUFACTURER" "Panasonic Electronic Components" (id 5) (at 85.09 86.36 0)
+      (effects (font (size 1.27 1.27)) hide)
+    )
+    (property "Manufacturer_Name" "Panasonic Electronic Components" (id 6) (at 85.09 86.36 0)
+      (effects (font (size 1.27 1.27)) hide)
+    )
+    (property "Manufacturer_Part_Number" "ERJ-6ENF1001V" (id 7) (at 85.09 86.36 0)
+      (effects (font (size 1.27 1.27)) hide)
+    )
+    (property "LCSC" "" (id 8) (at 85.09 86.36 0)
+      (effects (font (size 1.27 1.27)) hide)
+    )
+    (property "Digi-Key Part Number" "P1.00KCCT-ND" (id 9) (at 85.09 86.36 0)
+      (effects (font (size 1.27 1.27)) hide)
+    )
