File: board/swd.kicad_sch (KiCad schematic)
At the start: 1 part, among them J7 0702462004

Commit message: created firmware project. Tested MIDI communication over MIDI port as well as USB MIDI
Parts:
- J7: Digi-Key Part Number (none) -> WM3479-ND
Changed lines of the file:
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@@
+      (effects (font (size 1.27 1.27)) hide)
+    )
+    (property "Digi-Key Part Number" "WM3479-ND" (id 8) (at 91.44 80.01 0)
       (effects (font (size 1.27 1.27)) hide)
     )
