File: board/usbConn.kicad_sch (KiCad schematic)
At the start: 1 part, among them J6 292304-1

Commit message: created firmware project. Tested MIDI communication over MIDI port as well as USB MIDI
Parts:
- J6: Digi-Key Part Number (none) -> A31725-ND
Changed lines of the file:
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@@
+      (effects (font (size 1.27 1.27)) hide)
+    )
+    (property "Digi-Key Part Number" "A31725-ND" (id 14) (at 90.17 88.9 0)
       (effects (font (size 1.27 1.27)) hide)
     )
